File: simple/simple.kicad_sch (KiCad schematic)
At the start: 2 parts, among them J1 Screw_Terminal_01x02, U1 RPMH3.3-1.5

Commit message: adding power input led
Signed-off-by: Per Hallsmark <per@hallsmark.se>
Parts:
- added D1: LED, symbol Device:LED
- added R1: 4k7, symbol Device:R
Connections:
- net GND: now also D1.1 (K)
- net VCC: now also R1.1
- new net: D1.2 (A), R1.2
Changed lines of the file:
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@@
   (junction (at 36.83 100.33) (diameter 0) (color 0 0 0 0)
   )
+  (junction (at 50.8 100.33) (diameter 0) (color 0 0 0 0)
+  )
   (junction (at 36.83 78.74) (diameter 0) (color 0 0 0 0)
   )
+  (junction (at 50.8 78.74) (diameter 0) (color 0 0 0 0)
+  )
   (junction (at 77.47 100.33) (diameter 0) (color 0 0 0 0)
   )
+  (wire (pts (xy 50.8 87.63) (xy 50.8 90.17))
+    (stroke (width 0) (type default))
+  )
+  (wire (pts (xy 50.8 78.74) (xy 50.8 80.01))
+    (stroke (width 0) (type default))
+  )
   (wire (pts (xy 77.47 100.33) (xy 99.06 100.33))
     (stroke (width 0) (type default))
   )
-  (wire (pts (xy 36.83 78.74) (xy 67.31 78.74))
+  (wire (pts (xy 50.8 97.79) (xy 50.8 100.33))
+    (stroke (width 0) (type default))
+  )
+  (wire (pts (xy 36.83 78.74) (xy 50.8 78.74))
+    (stroke (width 0) (type default))
+  )
+  (wire (pts (xy 50.8 100.33) (xy 77.47 100.33))
     (stroke (width 0) (type default))
   )
@@
     (stroke (width 0) (type default))
   )
-  (wire (pts (xy 36.83 100.33) (xy 77.47 100.33))
+  (wire (pts (xy 36.83 100.33) (xy 50.8 100.33))
+    (stroke (width 0) (type default))
+  )
+  (wire (pts (xy 50.8 78.74) (xy 67.31 78.74))
     (stroke (width 0) (type default))
   )
@@
     )
   )
+  (symbol (lib_id "Device:R") (at 50.8 83.82 0) (unit 1)
+    (in_bom yes) (on_board yes) (dnp no) (fields_autoplaced)
+    (property "Reference" "R1" (at 53.34 82.55 0)
+      (effects (font (size 1.27 1.27)) (justify left))
+    )
+    (property "Value" "4k7" (at 53.34 85.09 0)
+      (effects (font (size 1.27 1.27)) (justify left))
+    )
+    (property "Footprint" "" (at 49.022 83.82 90)
+      (effects (font (size 1.27 1.27)) hide)
+    )
+    (property "Datasheet" "~" (at 50.8 83.82 0)
+      (effects (font (size 1.27 1.27)) hide)
+    )
+    (pin "1")
+    (pin "2")
+    (instances
+      (project "simple"
+        (path "/811f7822-4cec-430f-a1d6-2c346407fe4c"
+          (reference "R1") (unit 1)
+        )
+      )
+    )
+  )
   (symbol (lib_id "power:VCC") (at 36.83 78.74 0) (unit 1)
     (in_bom yes) (on_board yes) (dnp no) (fields_autoplaced)
@@
         )
       )
+    )
+  )
+  (symbol (lib_id "Device:LED") (at 50.8 93.98 90) (unit 1)
+    (in_bom yes) (on_board yes) (dnp no) (fields_autoplaced)
+    (property "Reference" "D1" (at 54.61 94.2975 90)
+      (effects (font (size 1.27 1.27)) (justify right))
+    )
+    (property "Value" "LED" (at 54.61 96.8375 90)
+      (effects (font (size 1.27 1.27)) (justify right))
+    )
+    (property "Footprint" "" (at 50.8 93.98 0)
+      (effects (font (size 1.27 1.27)) hide)
+    )
+    (property "Datasheet" "~" (at 50.8 93.98 0)
+      (effects (font (size 1.27 1.27)) hide)
+    )
+    (pin "1")
+    (pin "2")
+    (instances
+      (project "simple"
+        (path "/811f7822-4cec-430f-a1d6-2c346407fe4c"
+          (reference "D1") (unit 1)
+        )
+      )
